File: Shield_Emergent_4.kicad_sch (KiCad schematic)
At the start: 33 parts, among them J1 TF31-18S-0.5SH_800_, J2 Conn_01x04_Socket, J3 TF31-18S-0.5SH_800_, J4 Conn_01x05, J5 Conn_01x02_Socket, J6 Conn_01x02_Socket, J7 Conn_01x05, J8 Conn_02x05_Odd_Even, U3 SP3012-06UTG, U4 SP3012-06UTG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

Commit message: v0.2 Draft routing
Parts:
- J8: footprint Connector_PinHeader_1.27mm:PinHeader_2x05_P1.27mm_Vertical -> myLib8:DS1020-04-10BVT1
Changed lines of the file:
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@@
 			)
 		)
-		(property "Footprint" "Connector_PinHeader_1.27mm:PinHeader_2x05_P1.27mm_Vertical"
+		(property "Footprint" "myLib8:DS1020-04-10BVT1"
 			(at 158.75 127 0)
 			(effects
